File: FMCW/tx.kicad_pcb (KiCad board)
At the start: 2 copper layers, 66 parts, among them J1 Barrel_Jack, J2 SMA_RX, J3 SMA_TX, U1 ADF4158, U10 HMC431LP4, U2 LM1117-3.3, U3 TLV172DCK, U4 LP2985-5.0, U5 LP2985-10.0, U6 LP2985-3.0, U7 SE5003_1

Commit message: Updated Files
Parts:
- added J4: Conn_01x07_Male, Pin_Headers:Pin_Header_Straight_1x07_Pitch2.54mm, F.Cu at (94.2, 90.7)
- moved U2 78.2 mm to (85.9, 83.1), turned to 180 degrees
- moved C1 75.3 mm to (78.5, 106.2), turned to 180 degrees
- moved C13 70.6 mm to (78.5, 114.3), turned to 180 degrees
- moved C12 70.4 mm to (78.5, 112.0), turned to 180 degrees
- moved C9 66.2 mm to (78.5, 109.7), turned to 180 degrees
- moved C15 65.3 mm to (83.8, 114.3)
- moved C16 65.1 mm to (83.8, 112.0)
- moved L1 65.0 mm to (83.6, 107.7), turned to 90 degrees
- moved C17 59.0 mm to (93.2, 84.3), turned to 270 degrees
- moved J1 58.5 mm to (81.3, 102.1), turned to 270 degrees
- moved C18 53.9 mm to (95.2, 113.0), turned to 270 degrees
- moved C19 46.3 mm to (103.4, 115.3), turned to 270 degrees
- moved C4 44.9 mm to (103.9, 100.3)
- moved C5 44.7 mm to (103.9, 102.4)
- moved C43 44.6 mm to (103.9, 104.4)
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Connections:
- U1 pad 12: /ADC_TXDATA -> Net-(J4-Pad4)
- U1 pad 13: /ADF_CE -> Net-(J4-Pad3)
- U1 pad 14: /ADC_CLK -> Net-(J4-Pad5)
- U1 pad 15: /ADC_DATA -> Net-(J4-Pad6)
- U1 pad 16: /ADF_LE -> Net-(J4-Pad7)
- U1 pad 17: /MUXOUT -> Net-(J4-Pad2)
- U1 pad 9: /REFIN -> Net-(J4-Pad1)

Commit message: Updated Files
Parts:
- moved C17 7.62 mm to (100.8, 84.3)
- moved U2 7.62 mm to (93.5, 83.1)
- moved U7 0.25 mm to (156.5, 97.5)
Changed lines of the file:
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@@
 (kicad_pcb (version 4) (host pcbnew 4.0.7)
   (general
-    (links 184)
-    (no_connects 158)
-    (area 182.895142 16.51 276.007905 59.89)
+    (links 194)
+    (no_connects 159)
+    (area 74.304999 77.583 188.153 117.341001)
     (thickness 1.6)
     (drawings 0)
@@
   )
   (setup
-    (last_trace_width 2.951275)
+    (last_trace_width 0.25)
     (user_trace_width 0.3)
-    (user_trace_width 1)
+    (user_trace_width 1.4718)
     (user_trace_width 2.951275)
     (trace_clearance 0.2)
@@
     (mod_text_size 1 1)
     (mod_text_width 0.15)
-    (pad_size 1.5 1.5)
-    (pad_drill 0.6)
+    (pad_size 2.5 2.5)
+    (pad_drill 0)
     (pad_to_mask_clearance 0)
     (aux_axis_origin 0 0)
@@
     (add_net "Net-(U7-Pad7)")
   )
+  (module fmcw:SE5003 (layer F.Cu)
+    (at 156.464 97.536)
+    (fp_text reference U7 (at -0.03 3.1) (layer F.SilkS)
+      (effects (font (size 1 1) (thickness 0.15)))
+    )
+    (fp_text value SE5003_1 (at 0.06 -3.11) (layer F.Fab)
+      (effects (font (size 1 1) (thickness 0.15)))
+    )
+    (fp_line (start -2 -1.61) (end -1.61 -2) (layer F.SilkS) (width 0.15))
+    (fp_line (start -2 2) (end 2 2) (layer F.SilkS) (width 0.15))
+    (fp_line (start 2 -2) (end 2 2) (layer F.SilkS) (width 0.15))
+    (fp_line (start -1.6 -2) (end 2 -2) (layer F.SilkS) (width 0.15))
+    (fp_line (start -2 2) (end -2 -1.6) (layer F.SilkS) (width 0.15))
+    (fp_line (start -1.6 2) (end 1.6 2) (layer F.SilkS) (width 0.15))
+    (pad 1 smd rect (at -1.85 -1 90) (size 0.35 0.8) (layers F.Cu F.Paste F.Mask)
+      (net 32 "Net-(U7-Pad1)"))
+    (pad 2 smd rect (at -1.85 -0.5 90) (size 0.35 0.8) (layers F.Cu F.Paste F.Mask)
+      (net 2 GND))
+    (pad 3 smd rect (at -1.85 0 90) (size 0.35 0.8) (layers F.Cu F.Paste F.Mask)
+      (net 30 "Net-(R11-Pad1)"))
+    (pad 4 smd rect (at -1.85 0.5 90) (size 0.35 0.8) (layers F.Cu F.Paste F.Mask)
+      (net 2 GND))
+    (pad 5 smd rect (at -1.85 1 90) (size 0.35 0.8) (layers F.Cu F.Paste F.Mask)
+      (net 19 "Net-(C37-Pad2)"))
+    (pad 15 smd rect (at 1.85 -1 90) (size 0.35 0.8) (layers F.Cu F.Paste F.Mask)
+      (net 2 GND))
+    (pad 14 smd rect (at 1.85 -0.5 90) (size 0.35 0.8) (layers F.Cu F.Paste F.Mask)
+      (net 2 GND))
+    (pad 13 smd rect (at 1.85 0 90) (size 0.35 0.8) (layers F.Cu F.Paste F.Mask)
+      (net 25 "Net-(R3-Pad2)"))
+    (pad 12 smd rect (at 1.85 0.5 90) (size 0.35 0.8) (layers F.Cu F.Paste F.Mask)
+      (net 2 GND))
+    (pad 11 smd rect (at 1.85 1 90) (size 0.35 0.8) (layers F.Cu F.Paste F.Mask)
+      (net 2 GND))
+    (pad 8 smd rect (at 0 1.85) (size 0.35 0.8) (layers F.Cu F.Paste F.Mask)
+      (net 19 "Net-(C37-Pad2)"))
+    (pad 9 smd rect (at 0.5 1.85) (size 0.35 0.8) (layers F.Cu F.Paste F.Mask)
+      (net 19 "Net-(C37-Pad2)"))
+    (pad 10 smd rect (at 1 1.85) (size 0.35 0.8) (layers F.Cu F.Paste F.Mask)
+      (net 33 "Net-(U7-Pad10)"))
+    (pad 7 smd rect (at -0.5 1.85) (size 0.35 0.8) (layers F.Cu F.Paste F.Mask)
+      (net 34 "Net-(U7-Pad7)"))
+    (pad 6 smd rect (at -1 1.85) (size 0.35 0.8) (layers F.Cu F.Paste F.Mask)
+      (net 35 "Net-(U7-Pad6)"))
+    (pad 20 smd rect (at -1 -1.85) (size 0.35 0.8) (layers F.Cu F.Paste F.Mask)
+      (net 19 "Net-(C37-Pad2)"))
+    (pad 19 smd rect (at -0.5 -1.85) (size 0.35 0.8) (layers F.Cu F.Paste F.Mask)
+      (net 19 "Net-(C37-Pad2)"))
+    (pad 18 smd rect (at 0 -1.85) (size 0.35 0.8) (layers F.Cu F.Paste F.Mask)
+      (net 19 "Net-(C37-Pad2)"))
+    (pad 17 smd rect (at 0.5 -1.85) (size 0.35 0.8) (layers F.Cu F.Paste F.Mask)
+      (net 2 GND))
+    (pad 16 smd rect (at 1 -1.85) (size 0.35 0.8) (layers F.Cu F.Paste F.Mask)
+      (net 2 GND))
+    (pad 2 smd rect (at 0 0) (size 2.35 2.35) (layers F.Cu F.Paste F.Mask)
+      (net 2 GND))
+    (pad 2 thru_hole circle (at -0.67 -0.67) (size 0.27 0.27) (drill 0.25) (layers *.Cu *.Mask)
+      (net 2 GND))
+    (pad 2 thru_hole circle (at 0 -0.67) (size 0.27 0.27) (drill 0.25) (layers *.Cu *.Mask)
+      (net 2 GND))
+    (pad 2 thru_hole circle (at 0.67 -0.67) (size 0.27 0.27) (drill 0.25) (layers *.Cu *.Mask)
+      (net 2 GND))
+    (pad 2 thru_hole circle (at -0.67 0) (size 0.27 0.27) (drill 0.25) (layers *.Cu *.Mask)
+      (net 2 GND))
+    (pad 2 thru_hole circle (at 0 0) (size 0.27 0.27) (drill 0.25) (layers *.Cu *.Mask)
+      (net 2 GND))
+    (pad 2 thru_hole circle (at 0.67 0) (size 0.27 0.27) (drill 0.25) (layers *.Cu *.Mask)
+      (net 2 GND))
+    (pad 2 thru_hole circle (at -0.67 0.67) (size 0.27 0.27) (drill 0.25) (layers *.Cu *.Mask)
+      (net 2 GND))
+    (pad 2 thru_hole circle (at 0 0.67) (size 0.27 0.27) (drill 0.25) (layers *.Cu *.Mask)
+      (net 2 GND))
+    (pad 2 thru_hole circle (at 0.67 0.67) (size 0.27 0.27) (drill 0.25) (layers *.Cu *.Mask)
+      (net 2 GND))
+  )
   (module Capacitors_SMD:C_0805_HandSoldering (layer F.Cu)
     (at 78.486 106.172 180)
@@
   )
   (module Capacitors_SMD:C_0805_HandSoldering (layer F.Cu)
-    (at 93.218 84.328 270)
+    (at 100.838 84.328 270)
     (descr "Capacitor SMD 0805, hand soldering")
     (tags "capacitor 0805")
@@
   )
   (module TO_SOT_Packages_SMD:TO-252-3_TabPin2 (layer F.Cu)
-    (at 85.852 83.058 180)
+    (at 93.472 83.058 180)
     (descr "TO-252 / DPAK SMD package, http://www.infineon.com/cms/en/product/packages/PG-TO252/PG-TO252-3-1/")
     (tags "DPAK TO-252 DPAK-3 TO-252-3 SOT-428")
@@
     )
   )
-  (module fmcw:SE5003 (layer F.Cu)
-    (at 156.21 97.536)
-    (fp_text reference U7 (at -0.03 3.1) (layer F.SilkS)
-      (effects (font (size 1 1) (thickness 0.15)))
-    )
-    (fp_text value SE5003_1 (at 0.06 -3.11) (layer F.Fab)
-      (effects (font (size 1 1) (thickness 0.15)))
-    )
-    (fp_line (start -2 -1.61) (end -1.61 -2) (layer F.SilkS) (width 0.15))
-    (fp_line (start -2 2) (end 2 2) (layer F.SilkS) (width 0.15))
-    (fp_line (start 2 -2) (end 2 2) (layer F.SilkS) (width 0.15))
-    (fp_line (start -1.6 -2) (end 2 -2) (layer F.SilkS) (width 0.15))
-    (fp_line (start -2 2) (end -2 -1.6) (layer F.SilkS) (width 0.15))
-    (fp_line (start -1.6 2) (end 1.6 2) (layer F.SilkS) (width 0.15))
-    (pad 1 smd rect (at -1.85 -1 90) (size 0.35 0.8) (layers F.Cu F.Paste F.Mask)
-      (net 32 "Net-(U7-Pad1)"))
-    (pad 2 smd rect (at -1.85 -0.5 90) (size 0.35 0.8) (layers F.Cu F.Paste F.Mask)
-      (net 2 GND))
-    (pad 3 smd rect (at -1.85 0 90) (size 0.35 0.8) (layers F.Cu F.Paste F.Mask)
-      (net 30 "Net-(R11-Pad1)"))
-    (pad 4 smd rect (at -1.85 0.5 90) (size 0.35 0.8) (layers F.Cu F.Paste F.Mask)
-      (net 2 GND))
-    (pad 5 smd rect (at -1.85 1 90) (size 0.35 0.8) (layers F.Cu F.Paste F.Mask)
-      (net 19 "Net-(C37-Pad2)"))
-    (pad 15 smd rect (at 1.85 -1 90) (size 0.35 0.8) (layers F.Cu F.Paste F.Mask)
-      (net 2 GND))
-    (pad 14 smd rect (at 1.85 -0.5 90) (size 0.35 0.8) (layers F.Cu F.Paste F.Mask)
-      (net 2 GND))
-    (pad 13 smd rect (at 1.85 0 90) (size 0.35 0.8) (layers F.Cu F.Paste F.Mask)
-      (net 25 "Net-(R3-Pad2)"))
-    (pad 12 smd rect (at 1.85 0.5 90) (size 0.35 0.8) (layers F.Cu F.Paste F.Mask)
-      (net 2 GND))
-    (pad 11 smd rect (at 1.85 1 90) (size 0.35 0.8) (layers F.Cu F.Paste F.Mask)
-      (net 2 GND))
-    (pad 8 smd rect (at 0 1.85) (size 0.35 0.8) (layers F.Cu F.Paste F.Mask)
-      (net 19 "Net-(C37-Pad2)"))
-    (pad 9 smd rect (at 0.5 1.85) (size 0.35 0.8) (layers F.Cu F.Paste F.Mask)
-      (net 19 "Net-(C37-Pad2)"))
-    (pad 10 smd rect (at 1 1.85) (size 0.35 0.8) (layers F.Cu F.Paste F.Mask)
-      (net 33 "Net-(U7-Pad10)"))
-    (pad 7 smd rect (at -0.5 1.85) (size 0.35 0.8) (layers F.Cu F.Paste F.Mask)
-      (net 34 "Net-(U7-Pad7)"))
-    (pad 6 smd rect (at -1 1.85) (size 0.35 0.8) (layers F.Cu F.Paste F.Mask)
-      (net 35 "Net-(U7-Pad6)"))
-    (pad 20 smd rect (at -1 -1.85) (size 0.35 0.8) (layers F.Cu F.Paste F.Mask)
-      (net 19 "Net-(C37-Pad2)"))
-    (pad 19 smd rect (at -0.5 -1.85) (size 0.35 0.8) (layers F.Cu F.Paste F.Mask)
-      (net 19 "Net-(C37-Pad2)"))
-    (pad 18 smd rect (at 0 -1.85) (size 0.35 0.8) (layers F.Cu F.Paste F.Mask)
-      (net 19 "Net-(C37-Pad2)"))
-    (pad 17 smd rect (at 0.5 -1.85) (size 0.35 0.8) (layers F.Cu F.Paste F.Mask)
-      (net 2 GND))
-    (pad 16 smd rect (at 1 -1.85) (size 0.35 0.8) (layers F.Cu F.Paste F.Mask)
-      (net 2 GND))
-    (pad 0 smd rect (at 0 0) (size 2.35 2.35) (layers F.Cu F.Paste F.Mask))
-  )
   (module fmcw3:VQFN-24 (layer F.Cu)

Commit message: Updated Files
Parts:
- removed C214, C215, C37: DNP, Capacitors_SMD:C_0805_HandSoldering
- added C32: 750p, Capacitors_SMD:C_0603_HandSoldering, F.Cu at (239.8, 117.7)
- added C33: 100n, Capacitors_SMD:C_0603_HandSoldering, F.Cu at (202.9, 152.4)
- added C34: 100n, Capacitors_SMD:C_0603_HandSoldering, F.Cu at (219.1, 136.5)
- added C35: 56n, Capacitors_SMD:C_0603_HandSoldering, F.Cu at (235.7, 117.7)
- added R13: 226, Resistors_SMD:R_0805_HandSoldering, F.Cu at (226.0, 112.7)
- added R14: 10, Resistors_SMD:R_0805_HandSoldering, F.Cu at (236.3, 112.7)
- added U8: TCXO, buradar:TCXO, F.Cu at (220.2, 113.8)
- C1, C12, C13, C15, C16, C38, C9: footprint Capacitors_SMD:C_0805_HandSoldering -> Capacitors_SMD:C_0603_HandSoldering
- C10: value 2.2n -> 1u
- C11, C8: value 10p -> 100p
- C14: value 56p -> 47p
- C17: value 10u -> 10n; footprint Capacitors_SMD:C_0805_HandSoldering -> Capacitors_SMD:C_0603_HandSoldering
- C18: value 1u -> 10u
- C19: value 10n -> 4.7u
- C20: value 10u -> 100u
- C24, C26, C30: value 10u -> 4.7u; footprint Capacitors_SMD:C_0805_HandSoldering -> Capacitors_SMD:C_0603_HandSoldering
- C29: value 47p -> 20n
- C31: value 22p -> 10n
- J2, J3: footprint fmcw:SMA -> buradar:SMA
- J4: value Conn_01x07_Male -> Conn_01x06_Male; footprint Pin_Headers:Pin_Header_Straight_1x07_Pitch2.54mm -> Pin_Headers:Pin_Header_Straight_1x06_Pitch2.54mm
- R2: value DNP -> 1.02k
- R5: value 4.7k -> 1.1k
- R6: value 4.7k -> 3.74k
- R7: value 4.7k -> 5k
- U1: footprint fmcw3:VFQFN-24 -> buradar:VFQFN-24
- U10: footprint fmcw3:VQFN-24 -> buradar:VQFN-24
- U2: value LM1117-3.3 -> LP2985-3.3; footprint TO_SOT_Packages_SMD:TO-252-3_TabPin2 -> TO_SOT_Packages_SMD:SOT-23-5_HandSoldering
- U4: value LP2985-5.0 -> LM1117-5.0; footprint TO_SOT_Packages_SMD:SOT-23-5_HandSoldering -> TO_SOT_Packages_SMD:TO-252-3_TabPin2
- U7: footprint fmcw:SE5003 -> buradar:SE5003
- moved C12 160.4 mm to (237.6, 132.1), turned to 0 degrees
- moved C13 156.3 mm to (233.6, 133.5), turned to 0 degrees
- moved C18 152.8 mm to (248.0, 117.0), turned to 0 degrees
- moved C9 149.5 mm to (224.0, 143.8), turned to 0 degrees
- moved C17 147.9 mm to (243.9, 121.8), turned to 0 degrees
- moved C5 144.8 mm to (246.7, 126.6)
- moved C4 142.2 mm to (242.7, 131.4)
- moved C16 140.4 mm to (220.0, 146.1)
- moved C15 136.3 mm to (215.1, 150.9)
- moved C7 135.9 mm to (242.6, 126.6), turned to 0 degrees
- moved C8 134.7 mm to (248.0, 121.8), turned to 0 degrees
- moved C6 130.9 mm to (237.7, 136.9), turned to 0 degrees
- moved C19 130.8 mm to (233.4, 128.7), turned to 0 degrees
- moved C21 130.1 mm to (249.0, 112.2), turned to 0 degrees
- moved C1 128.9 mm to (198.8, 152.4), turned to 0 degrees
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Connections:
- C10 pad 1: Net-(C10-Pad1) -> /12V
- C10 pad 2: Net-(C10-Pad2) -> GND
- C14 pad 1: Net-(C10-Pad1) -> Net-(C14-Pad1)
- C14 pad 2: GND -> Net-(C14-Pad2)
- C17 pad 1: /3V3 -> Net-(C17-Pad1)
- C19 pad 1: Net-(C19-Pad1) -> /3V3
- C29 pad 2: GND -> Net-(C29-Pad2)
- C31 pad 1: Net-(C29-Pad1) -> Net-(C31-Pad1)
- C38 pad 2: Net-(C37-Pad2) -> Net-(C38-Pad2)
- C39 pad 2: Net-(C37-Pad2) -> Net-(C38-Pad2)
- C40 pad 2: Net-(C37-Pad2) -> Net-(C38-Pad2)
- C41 pad 2: Net-(C37-Pad2) -> Net-(C38-Pad2)
- L4 pad 1: Net-(C37-Pad2) -> Net-(C38-Pad2)
- L4 pad 2: /3V3 -> /5V
- R2 pad 1: Net-(C10-Pad2) -> Net-(C14-Pad2)
- R4 pad 1: Net-(C10-Pad2) -> Net-(C14-Pad2)
- R5 pad 1: Net-(R5-Pad1) -> Net-(C32-Pad2)
- R5 pad 2: GND -> Net-(C14-Pad1)
- R6 pad 1: Net-(R6-Pad1) -> Net-(C31-Pad1)
- R6 pad 2: Net-(R5-Pad1) -> /5V
- R7 pad 1: Net-(C29-Pad1) -> Net-(C31-Pad1)
- R7 pad 2: Net-(R6-Pad1) -> GND
- U1 pad 12: Net-(J4-Pad4) -> Net-(J4-Pad3)
- U1 pad 13: Net-(J4-Pad3) -> Net-(J4-Pad2)
- U1 pad 14: Net-(J4-Pad5) -> Net-(J4-Pad4)
- U1 pad 15: Net-(J4-Pad6) -> Net-(J4-Pad5)
- U1 pad 16: Net-(J4-Pad7) -> Net-(J4-Pad6)
- U1 pad 17: Net-(J4-Pad2) -> Net-(J4-Pad1)
- U1 pad 24: Net-(C10-Pad1) -> Net-(C14-Pad1)
- U1 pad 9: Net-(J4-Pad1) -> Net-(C34-Pad2)
- U10 pad 22: Net-(C29-Pad1) -> Net-(C35-Pad1)
- U2 pad 1: GND -> /12V
- U2 pad 2: /3V3 -> GND
- U3 pad 1: Net-(R6-Pad1) -> Net-(C29-Pad1)
- U3 pad 3: Net-(C10-Pad1) -> GND
- U3 pad 4: Net-(R5-Pad1) -> Net-(C32-Pad2)
- U4 pad 1: /12V -> GND
- U4 pad 2: GND -> /5V
- U7 pad 18: Net-(C37-Pad2) -> Net-(C38-Pad2)
- U7 pad 19: Net-(C37-Pad2) -> Net-(C38-Pad2)
- U7 pad 20: Net-(C37-Pad2) -> Net-(C38-Pad2)
- U7 pad 5: Net-(C37-Pad2) -> Net-(C31-Pad1)
- U7 pad 8: Net-(C37-Pad2) -> Net-(C38-Pad2)
- U7 pad 9: Net-(C37-Pad2) -> Net-(C38-Pad2)

Commit message: Updated BOM
Parts:
- added D1: LED, LEDs:LED_0805_HandSoldering, F.Cu at (0.00, 0.00)
- added R15: 1k, Resistors_SMD:R_0805_HandSoldering, F.Cu at (0.00, 0.00)
- added R16: 10k, Resistors_SMD:R_0805_HandSoldering, F.Cu at (0.00, 0.00)
- C12: value 10u -> 100u
- C9: value 10u -> 470u
- moved C6 102.0 mm to (269.2, 39.9)
- moved C13 102.0 mm to (265.0, 36.5)
- moved C16 102.0 mm to (251.5, 49.1)
- moved C25 102.0 mm to (238.5, 54.0)
- moved C30 102.0 mm to (243.3, 48.5)
- moved C40 102.0 mm to (247.4, 49.1)
- moved C41 102.0 mm to (254.8, 42.0)
- moved J4 102.0 mm to (209.5, 16.3)
- moved R1 102.0 mm to (251.1, 34.4)
- moved R10 102.0 mm to (251.1, 23.4)
- moved R8 102.0 mm to (251.1, 28.9)
- moved U1 102.0 mm to (234.1, 24.8)
- moved U4 102.0 mm to (222.5, 51.3)
- moved U8 102.0 mm to (251.7, 16.7)
- moved C1 102.0 mm to (230.3, 55.4)
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Connections:
- C1 pad 2: GND -> Net-(C1-Pad2)
- C12 pad 1: /12V -> /5V
- C9 pad 1: /12V -> Net-(C9-Pad1)
- C9 pad 2: GND -> Net-(C9-Pad2)
- J1 pad 2: GND -> Net-(J1-Pad2)
- J1 pad 3: GND -> Net-(J1-Pad2)
- L1 pad 1: /12V -> Net-(L1-Pad1)
- U7 pad GND: GND -> (no net)

Commit message: Updated pcb files
Parts:
- removed C13, C15, C16, C18: 10u, Capacitors_SMD:C_0603_HandSoldering
- removed C20: 100u, Capacitors_SMD:C_0805_HandSoldering
- added R17: 510, Resistors_SMD:R_0805_HandSoldering, F.Cu at (162.6, 110.7)
- C1, C12: footprint Capacitors_SMD:C_0603_HandSoldering -> Capacitors_SMD:C_1206_HandSoldering
- C24: value 4.7u -> 2.2u
- C9: footprint Capacitors_SMD:C_0603_HandSoldering -> Capacitors_SMD:CP_Elec_10x10
- J2, J3: footprint buradar:SMA -> buradar:SMA_molex_straight
- R1: value 5.49k -> 5.1k
- R11, R12, R9: value 18 -> 16
- R13: value 226 -> 220
- R5: value 1.1k -> 1k
- R6: value 3.74k -> 3.3k
- R7: value 5k -> 5.1k
- moved C9 200.0 mm to (71.1, 124.2)
- moved L1 189.1 mm to (78.5, 115.3)
- moved C17 188.9 mm to (109.7, 115.6), turned to 180 degrees
- moved C5 188.8 mm to (108.0, 111.3), turned to 180 degrees
- moved C8 183.6 mm to (112.3, 100.6), turned to 180 degrees
- moved C4 182.5 mm to (108.0, 109.7), turned to 180 degrees
- moved C19 180.1 mm to (106.9, 118.1), turned to 270 degrees
- moved C7 179.9 mm to (115.3, 114.0)
- moved C21 175.0 mm to (128.8, 102.4)
- moved C6 171.4 mm to (115.3, 115.6)
- moved C32 171.0 mm to (126.7, 112.0), turned to 270 degrees
- moved C43 171.0 mm to (108.0, 112.8), turned to 180 degrees
- moved R14 167.8 mm to (128.5, 109.2), turned to 180 degrees
- moved C3 165.8 mm to (103.9, 103.9), turned to 90 degrees
- moved U8 165.6 mm to (102.1, 87.6)
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Connections:
- C1 pad 1: Net-(C1-Pad1) -> /12V
- C1 pad 2: Net-(C1-Pad2) -> GND
- C9 pad 1: Net-(C9-Pad1) -> /12V
- C9 pad 2: Net-(C9-Pad2) -> GND
- J1 pad 1: Net-(C1-Pad1) -> Net-(J1-Pad1)
- J1 pad 2: Net-(J1-Pad2) -> GND
- J1 pad 3: Net-(J1-Pad2) -> GND
- L1 pad 1: Net-(L1-Pad1) -> /12V
- L1 pad 2: Net-(C1-Pad1) -> Net-(J1-Pad1)
- R6 pad 1: Net-(C31-Pad1) -> Net-(R17-Pad2)
Routing:
- net GND: track 0.00 -> 61.5 mm
- net Net-(C38-Pad2): track 0.00 -> 34.4 mm
- net Net-(J2-Pad1): track 0.00 -> 33.4 mm
- net Net-(J3-Pad1): track 0.00 -> 33.0 mm
- net /5V: track 0.00 -> 21.5 mm
- net Net-(C31-Pad1): track 0.00 -> 10.6 mm
- net Net-(R10-Pad2): track 0.00 -> 9.77 mm
- net Net-(R9-Pad2): track 0.00 -> 9.31 mm
- net Net-(R11-Pad1): track 0.00 -> 8.74 mm
- net Net-(R11-Pad2): track 0.00 -> 8.31 mm
- net Net-(R3-Pad2): track 0.00 -> 6.20 mm
- net /12V: track 0.00 -> 3.40 mm
- net Net-(R17-Pad2): track 0.00 -> 2.03 mm

Commit message: Updated pcb files
Parts:
- moved C9 58.8 mm to (119.6, 90.9)
- moved L1 40.1 mm to (109.5, 89.9), turned to 180 degrees
- moved J1 35.1 mm to (103.9, 90.4), turned to 0 degrees
- moved U8 31.8 mm to (103.6, 119.4), turned to 270 degrees
- moved C33 31.8 mm to (103.6, 123.4), turned to 180 degrees
- moved C34 28.3 mm to (100.1, 114.0), turned to 90 degrees
- moved C11 11.2 mm to (121.7, 97.5)
- moved C26 4.37 mm to (135.6, 106.4), turned to 90 degrees
- moved L3 3.42 mm to (133.3, 109.7), turned to 0 degrees
- moved C28 2.27 mm to (134.1, 106.4), turned to 90 degrees
- moved C4 1.37 mm to (108.5, 111.0)
- moved C43 1.37 mm to (108.5, 114.0)
- moved C5 1.37 mm to (108.5, 112.5)
- moved R2 0.76 mm to (112.5, 108.5), turned to 180 degrees
Routing:
- net GND: track 61.5 -> 473.5 mm, vias 0 -> 2
- net /12V: track 3.40 -> 177.7 mm, vias 0 -> 5
- net /5V: track 21.5 -> 81.5 mm
- net /3V3: track 0.00 -> 38.3 mm, vias 0 -> 2
- net Net-(C11-Pad1): track 0.00 -> 30.3 mm
- net Net-(J4-Pad1): track 0.00 -> 27.9 mm, vias 0 -> 1
- net Net-(C32-Pad2): track 0.00 -> 20.2 mm
- net Net-(C6-Pad1): track 0.00 -> 19.7 mm
- net Net-(C11-Pad2): track 0.00 -> 18.9 mm
- net Net-(J4-Pad5): track 0.00 -> 15.0 mm, vias 0 -> 1
- net Net-(C38-Pad2): track 34.4 -> 19.7 mm, vias 0 -> 2
- net Net-(J4-Pad6): track 0.00 -> 14.5 mm, vias 0 -> 1
- net Net-(J4-Pad2): track 0.00 -> 13.4 mm, vias 0 -> 1
- net Net-(J4-Pad4): track 0.00 -> 12.4 mm, vias 0 -> 1
- net Net-(C35-Pad1): track 0.00 -> 11.8 mm
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Other:
- board outline added: 125 x 45 mm
